File: key_prac.kicad_pcb (KiCad board)
At the start: 2 copper layers, 20 parts, among them SW1 SW_Push, SW2 SW_Push, SW3 SW_Push, SW4 SW_Push, SW5 SW_Push, SW6 SW_Push, SW7 SW_Push, SW8 SW_Push, SW9 SW_Push, U1 promicro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

Commit message: pcb
Parts:
- moved SW9 6.84 mm to (63.5, 118.1)
- moved D2 3.59 mm to (91.4, 118.1)
- moved D5 3.59 mm to (115.6, 118.1)
- moved U1 3.59 mm to (63.5, 95.2)
- moved D1 3.59 mm to (82.5, 92.7)
- moved D3 3.59 mm to (82.5, 143.5)
- moved D4 3.59 mm to (104.1, 92.7)
- moved D6 3.59 mm to (118.1, 143.5)
- moved D7 3.59 mm to (125.7, 92.7)
- moved D8 3.59 mm to (134.6, 118.1)
- moved SW1 3.59 mm to (90.2, 74.9)
- moved SW3 3.59 mm to (90.2, 125.7)
- moved SW4 3.59 mm to (111.8, 74.9)
- moved SW6 3.59 mm to (133.3, 74.9)
- moved SW8 3.59 mm to (133.3, 125.7)
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Routing:
- net GND: track 116.6 -> 0.00 mm
- net Net-(U1-Pad18): track 188.0 -> 170.3 mm
- net Net-(SW9-Pad1): track 46.2 -> 54.4 mm
- net col0: track 110.3 -> 106.6 mm
- net row1: track 97.8 -> 99.9 mm
- net Net-(U1-Pad17): track 101.7 -> 103.4 mm
- net row0: track 86.9 -> 87.7 mm
- added copper zone on F.Cu, net GND
- removed copper zone on B.Cu, net GND
Other:
- board outline added: 101.6 x 87.6 mm

Commit message: gb
Routing:
- net Net-(U1-Pad18): track 170.3 -> 89.8 mm, vias 0 -> 1
- net Net-(U1-Pad16): track 104.1 -> 91.0 mm
- net Net-(SW9-Pad1): track 54.4 -> 57.1 mm
- net Net-(U1-Pad17): track 103.4 -> 104.6 mm
- net row0: track 87.7 -> 86.9 mm
Other:
- board size 101.6 x 87.6 mm -> 100.3 x 87.6 mm
