File: key_prac.kicad_pcb (KiCad board)
At the start: 2 copper layers, 100.3 x 87.6 mm, 20 parts, among them SW1 SW_Push, SW2 SW_Push, SW3 SW_Push, SW4 SW_Push, SW5 SW_Push, SW6 SW_Push, SW7 SW_Push, SW8 SW_Push, SW9 SW_Push, U1 promicro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

Commit message: beta
Routing:
- net col0: track 106.6 -> 105.9 mm
- added copper zone on B.Cu, net GND
Changed lines of the file:
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@@
     (thickness 1.6)
     (drawings 4)
-    (tracks 159)
+    (tracks 158)
     (zones 0)
     (modules 20)
@@
   (segment (start 90.17 125.73) (end 99.06 116.84) (width 0.25) (layer F.Cu) (net 12))
   (segment (start 64.77 80.01) (end 69.85 74.93) (width 0.25) (layer B.Cu) (net 12))
-  (segment (start 63.5 80.01) (end 64.77 80.01) (width 0.25) (layer B.Cu) (net 12))
-  (segment (start 63.5 88.9) (end 63.5 80.01) (width 0.25) (layer B.Cu) (net 12))
   (segment (start 55.88 96.52) (end 63.5 88.9) (width 0.25) (layer B.Cu) (net 12))
   (segment (start 69.85 74.93) (end 90.17 74.93) (width 0.25) (layer B.Cu) (net 12))
+  (segment (start 64.77 87.63) (end 63.5 88.9) (width 0.25) (layer B.Cu) (net 12))
+  (segment (start 64.77 80.01) (end 64.77 87.63) (width 0.25) (layer B.Cu) (net 12))
   (segment (start 120.65 83.82) (end 120.65 100.33) (width 0.25) (layer F.Cu) (net 13))
   (segment (start 111.76 74.93) (end 120.65 83.82) (width 0.25) (layer F.Cu) (net 13))
@@
   (segment (start 81.224999 121.864999) (end 85.192001 125.832001) (width 0.25) (layer F.Cu) (net 19))
   (segment (start 88.162999 125.832001) (end 89.485999 127.155001) (width 0.25) (layer F.Cu) (net 19))
-  (segment (start 75.74999 115.38501) (end 75.74999 96.06999) (width 0.25) (layer F.Cu) (net 20))
-  (segment (start 87.766008 127.60501) (end 87.005997 126.844999) (width 0.25) (layer F.Cu) (net 20))
-  (segment (start 59.872999 118.631761) (end 59.872999 117.588239) (width 0.25) (layer F.Cu) (net 20))
-  (segment (start 75.74999 96.06999) (end 71.12 91.44) (width 0.25) (layer F.Cu) (net 20))
-  (segment (start 94.64499 127.60501) (end 87.766008 127.60501) (width 0.25) (layer F.Cu) (net 20))
-  (segment (start 103.306999 118.546999) (end 94.64499 127.209008) (width 0.25) (layer F.Cu) (net 20))
-  (segment (start 87.005997 126.844999) (end 74.774999 126.844999) (width 0.25) (layer F.Cu) (net 20))
-  (segment (start 108.132999 118.546999) (end 103.306999 118.546999) (width 0.25) (layer F.Cu) (net 20))
-  (segment (start 74.774999 126.844999) (end 70.820402 122.890402) (width 0.25) (layer F.Cu) (net 20))
-  (segment (start 63.049409 117.022999) (end 67.4964 121.46999) (width 0.25) (layer F.Cu) (net 20))
-  (segment (start 67.4964 121.46999) (end 69.66501 121.46999) (width 0.25) (layer F.Cu) (net 20))
-  (segment (start 70.820402 122.890402) (end 64.13164 122.890402) (width 0.25) (layer F.Cu) (net 20))
-  (segment (start 69.66501 121.46999) (end 75.74999 115.38501) (width 0.25) (layer F.Cu) (net 20))
-  (segment (start 109.22 119.634) (end 108.132999 118.546999) (width 0.25) (layer F.Cu) (net 20))
-  (segment (start 60.438239 117.022999) (end 63.049409 117.022999) (width 0.25) (layer F.Cu) (net 20))
-  (segment (start 64.13164 122.890402) (end 59.872999 118.631761) (width 0.25) (layer F.Cu) (net 20))
-  (segment (start 94.64499 127.209008) (end 94.64499 127.60501) (width 0.25) (layer F.Cu) (net 20))
-  (segment (start 59.872999 117.588239) (end 60.438239 117.022999) (width 0.25) (layer F.Cu) (net 20))
+  (segment (start 108.132999 118.546999) (end 109.22 119.634) (width 0.25) (layer F.Cu) (net 20))
+  (segment (start 63.049409 117.022999) (end 60.438239 117.022999) (width 0.25) (layer F.Cu) (net 20))
+  (segment (start 67.4964 121.46999) (end 63.049409 117.022999) (width 0.25) (layer F.Cu) (net 20))
+  (segment (start 71.12 91.44) (end 75.74999 96.06999) (width 0.25) (layer F.Cu) (net 20))
+  (segment (start 69.66501 121.46999) (end 67.4964 121.46999) (width 0.25) (layer F.Cu) (net 20))
+  (segment (start 94.248988 127.60501) (end 103.306999 118.546999) (width 0.25) (layer F.Cu) (net 20))
+  (segment (start 75.74999 115.38501) (end 69.66501 121.46999) (width 0.25) (layer F.Cu) (net 20))
+  (segment (start 75.74999 96.06999) (end 75.74999 115.38501) (width 0.25) (layer F.Cu) (net 20))
+  (segment (start 59.872999 117.588239) (end 59.872999 118.631761) (width 0.25) (layer F.Cu) (net 20))
+  (segment (start 60.438239 117.022999) (end 59.872999 117.588239) (width 0.25) (layer F.Cu) (net 20))
+  (segment (start 59.872999 118.631761) (end 64.13164 122.890402) (width 0.25) (layer F.Cu) (net 20))
+  (segment (start 64.13164 122.890402) (end 70.820402 122.890402) (width 0.25) (layer F.Cu) (net 20))
+  (segment (start 70.820402 122.890402) (end 74.774999 126.844999) (width 0.25) (layer F.Cu) (net 20))
+  (segment (start 74.774999 126.844999) (end 87.005997 126.844999) (width 0.25) (layer F.Cu) (net 20))
+  (segment (start 87.005997 126.844999) (end 87.766008 127.60501) (width 0.25) (layer F.Cu) (net 20))
+  (segment (start 87.766008 127.60501) (end 94.248988 127.60501) (width 0.25) (layer F.Cu) (net 20))
+  (segment (start 103.306999 118.546999) (end 108.132999 118.546999) (width 0.25) (layer F.Cu) (net 20))
   (segment (start 71.12 93.98) (end 68.58 93.98) (width 0.25) (layer F.Cu) (net 21))
   (segment (start 64.952999 97.607001) (end 64.952999 109.402999) (width 0.25) (layer F.Cu) (net 21))
@@
       )
     )
+  )
+  (zone (net 15) (net_name GND) (layer B.Cu) (hatch edge 0.508)
+    (connect_pads (clearance 0.508))
+    (min_thickness 0.254)
+    (fill yes (arc_segments 32) (thermal_gap 0.508) (thermal_bridge_width 0.508))
+    (polygon
+      (pts
+        (xy 50.8 64.77) (xy 50.8 152.4) (xy 151.13 152.4) (xy 151.13 64.77)
+      )
+    )
